File: greenhouse/greenhouse.kicad_pcb (KiCad board)
At the start: 2 copper layers, 100 x 90 mm, 22 parts, among them J11 I2C-BME, J12 I2C-BME, J13 I2C-BME

Commit message: rework of PCB
Parts:
- renumbered Main5V to Main5V1
Connections:
- ESP32_DevKitV1 pad 1: Net-(ESP32_DevKitV1-Pad1) -> unconnected-(ESP32_DevKitV1-Pad1)
- ESP32_DevKitV1 pad 13: Motor1_Current -> Window2_closed
- ESP32_DevKitV1 pad 2: Window1_open -> Motor1_Current
- ESP32_DevKitV1 pad 24: SolarSense -> Window2_open
- ESP32_DevKitV1 pad 25: BatterySense -> Window1_closed
- ESP32_DevKitV1 pad 26: Motor2_Current -> Window1_open
- ESP32_DevKitV1 pad 3: Window1_closed -> Motor2_Current
- ESP32_DevKitV1 pad 33: Net-(ESP32_DevKitV1-Pad33) -> unconnected-(ESP32_DevKitV1-Pad33)
- ESP32_DevKitV1 pad 34: Net-(ESP32_DevKitV1-Pad34) -> unconnected-(ESP32_DevKitV1-Pad34)
- ESP32_DevKitV1 pad 4: Window2_open -> BatterySense
- ESP32_DevKitV1 pad 5: Window2_closed -> SolarSense
Routing:
- net Window1_open: track 31.5 -> 75.9 mm
- net Window2_open: track 25.4 -> 69.7 mm
- net Window1_closed: track 29.0 -> 72.9 mm
- net Motor2_Current: track 25.4 -> 65.4 mm
- net Motor1_Current: track 18.5 -> 58.4 mm, vias 0 -> 2
- net Window2_closed: track 21.0 -> 57.2 mm
- net BatterySense: track 29.1 -> 61.3 mm
- net SolarSense: track 32.2 -> 59.5 mm
- net 5V: track 260.9 -> 258.9 mm
- net GND: track 311.8 -> 310.7 mm
Other:
- outline, holes or cut-outs redrawn
- net class Default removed
